Commit message: renamed to mobina

File: mobina_description/urdf/mobina_calibration.xacro (robot description, xacro)
@@ -1,10 +1,10 @@
 <?xml version="1.0"?>
 <robot>
-  <property name="turtlebot_calib_cam_x" value="-0.0844382" />
-  <property name="turtlebot_calib_cam_y" value="0" />
-  <property name="turtlebot_calib_cam_z" value="0.1047496" />
-  <property name="turtlebot_calib_cam_rr" value="0" />
-  <property name="turtlebot_calib_cam_rp" value="0" />
-  <property name="turtlebot_calib_cam_ry" value="0" />
-  <property name="turtlebot_camera_parent_name" value="plate_2_link" />
+  <property name="mobina_calib_cam_x" value="0" />
+  <property name="mobina_calib_cam_y" value="0" />
+  <property name="mobina_calib_cam_z" value="0.105" />
+  <property name="mobina_calib_cam_rr" value="0" />
+  <property name="mobina_calib_cam_rp" value="0" />
+  <property name="mobina_calib_cam_ry" value="0" />
+  <property name="mobina_camera_parent_name" value="tray_base_link" />
 </robot>

File: mobina_description/urdf/mobina_hardware.urdf.xacro (robot description, xacro)
@@ -1,7 +1,7 @@
 <?xml version="1.0"?>
-<robot name="turtlebot_hardware" xmlns:xacro="http://ros.org/wiki/xacro">
+<robot name="mobina_hardware" xmlns:xacro="http://ros.org/wiki/xacro">
   <property name="M_PI" value="3.14159"/>
   <property name="M_SCALE" value="0.001"/>
-  <xacro:macro name="turtlebot_spacer" params="parent number x_loc y_loc z_loc">
+  <xacro:macro name="mobina_spacer" params="parent number x_loc y_loc z_loc">
     <joint name="spacer_${number}_joint" type="fixed">
       <origin xyz="${x_loc} ${y_loc} ${z_loc}" rpy="0 0 0" />
@@ -20,5 +20,5 @@
         <origin xyz=" 0 0 0 " rpy="0 0 0" />
         <geometry>
-          <mesh filename="package://turtlebot_description/meshes/68-02403-125_Spacer.dae" scale="${M_SCALE} ${M_SCALE} ${M_SCALE}"/>
+          <mesh filename="package://mobina_description/meshes/68-02403-125_Spacer.dae" scale="${M_SCALE} ${M_SCALE} ${M_SCALE}"/>
         </geometry>
       </visual>
@@ -31,5 +31,5 @@
     </link>
   </xacro:macro>
-  <xacro:macro name="turtlebot_standoff_1in" params="parent number x_loc y_loc z_loc">
+  <xacro:macro name="mobina_standoff_1in" params="parent number x_loc y_loc z_loc">
     <joint name="standoff_1in_${number}_joint" type="fixed">
       <origin xyz="${x_loc} ${y_loc} ${z_loc}" rpy="0 0 0" />
@@ -48,5 +48,5 @@
         <origin xyz=" 0 0 0 " rpy="0 0 0" />
         <geometry>
-          <mesh filename="package://turtlebot_description/meshes/68-04552-1000-RA_Turtlebot_M-F_Standoff.dae" scale="${M_SCALE} ${M_SCALE} ${M_SCALE}"/>
+          <mesh filename="package://mobina_description/meshes/68-04552-1000-RA_mobina_M-F_Standoff.dae" scale="${M_SCALE} ${M_SCALE} ${M_SCALE}"/>
         </geometry>
       </visual>
@@ -59,5 +59,5 @@
     </link>
   </xacro:macro>
-  <xacro:macro name="turtlebot_standoff_2in" params="parent number x_loc y_loc z_loc">
+  <xacro:macro name="mobina_standoff_2in" params="parent number x_loc y_loc z_loc">
     <joint name="standoff_2in_${number}_joint" type="fixed">
       <origin xyz="${x_loc} ${y_loc} ${z_loc}" rpy="0 0 0" />
@@ -76,5 +76,5 @@
         <origin xyz=" 0 0 0 " rpy="0 0 0" />
         <geometry>
-          <mesh filename="package://turtlebot_description/meshes/68-04552-2000-RA_Turtlebot_M-F_Standoff.dae" scale="${M_SCALE} ${M_SCALE} ${M_SCALE}"/>
+          <mesh filename="package://mobina_description/meshes/68-04552-2000-RA_mobina_M-F_Standoff.dae" scale="${M_SCALE} ${M_SCALE} ${M_SCALE}"/>
         </geometry>
       </visual>
@@ -87,5 +87,5 @@
     </link>
   </xacro:macro>
-  <xacro:macro name="turtlebot_standoff_8in" params="parent number x_loc y_loc z_loc">
+  <xacro:macro name="mobina_standoff_8in" params="parent number x_loc y_loc z_loc">
     <joint name="standoff_8in_${number}_joint" type="fixed">
       <origin xyz="${x_loc} ${y_loc} ${z_loc}" rpy="0 0 0" />
@@ -104,5 +104,5 @@
         <origin xyz=" 0 0 0 " rpy="0 0 0" />
         <geometry>
-          <mesh filename="package://turtlebot_description/meshes/68-02421-8000-RA_Turtlebot_F-F_Standoff.dae" scale="${M_SCALE} ${M_SCALE} ${M_SCALE}"/>
+          <mesh filename="package://mobina_description/meshes/68-02421-8000-RA_mobina_F-F_Standoff.dae" scale="${M_SCALE} ${M_SCALE} ${M_SCALE}"/>
         </geometry>
       </visual>
@@ -115,5 +115,5 @@
     </link>
   </xacro:macro>
-  <xacro:macro name="turtlebot_standoff_kinect" params="parent number x_loc y_loc z_loc">
+  <xacro:macro name="mobina_standoff_kinect" params="parent number x_loc y_loc z_loc">
     <joint name="standoff_kinect_${number}_joint" type="fixed">
       <origin xyz="${x_loc} ${y_loc} ${z_loc}" rpy="0 0 0" />
@@ -132,5 +132,5 @@
         <origin xyz=" 0 0 0 " rpy="0 0 0" />
         <geometry>
-          <mesh filename="package://turtlebot_description/meshes/68-04556-RA_Kinect_Standoff_Assy.3ds" scale="${M_SCALE} ${M_SCALE} ${M_SCALE}"/>
+          <mesh filename="package://mobina_description/meshes/68-04556-RA_Kinect_Standoff_Assy.3ds" scale="${M_SCALE} ${M_SCALE} ${M_SCALE}"/>
         </geometry>
       </visual>
