Commit message: renamed to mobina

File: mobina_description/urdf/mobina_body.urdf.xacro (robot description, xacro)
@@ -1,10 +1,10 @@
 <?xml version="1.0"?>
-<robot name="turtlebot_hardware" xmlns:xacro="http://ros.org/wiki/xacro">
+<robot name="mobina_hardware" xmlns:xacro="http://ros.org/wiki/xacro">
   <property name="M_PI" value="3.14159"/>
-  <!-- Macro for TurtleBot body. Including Gazebo extensions, but does not include Kinect -->
-  <include filename="$(find turtlebot_description)/urdf/gazebo.urdf.xacro"/>
+  <!-- Macro for mobina body. Including Gazebo extensions, but does not include Kinect -->
+  <include filename="$(find mobina_description)/urdf/gazebo.urdf.xacro"/>
   <property name="base_x" value="0.33" />
   <property name="base_y" value="0.33" />
-  <xacro:macro name="turtlebot_body">
+  <xacro:macro name="mobina_body">
     <material name="Green">
       <color rgba="0.0 0.8 0.0 1.0"/>
@@ -43,5 +43,5 @@
       <origin xyz=" 0 0 0.0308" rpy="0 0 0" />
       <geometry>
-        <mesh filename="package://turtlebot_description/meshes/create_body.dae"/>
+        <mesh filename="package://mobina_description/meshes/create_body.dae"/>
       </geometry>
     </visual>
@@ -61,4 +61,26 @@
     </inertial>
   </link>
+  <link name="tray_axis_link">
+    <inertial>
+      <mass value="0.01" />
+      <origin xyz="0 0 0"/>
+      <inertia ixx="0.001" ixy="0.0" ixz="0.0"
+        iyy="0.001" iyz="0.0" izz="0.001" />
+    </inertial>
+  </link>
+  <link name="tray_base_link">
+    <inertial>
+      <mass value="0.01" />
+      <origin xyz="0.035 0 0"/>
+      <inertia ixx="0.001" ixy="0.0" ixz="0.0"
+        iyy="0.001" iyz="0.0" izz="0.001" />
+    </inertial>
+  </link>
+  <joint name="tray_axis_joint" type="continuous">
+    <axis xyz="0 1 0"/>
+    <origin rpy="0 0 0" xyz="0 0 0"/>
+    <parent link="tray_axis_link"/>
+    <child link="tray_base_link"/>
+  </joint>
   <link name="left_cliff_sensor_link">
     <inertial>
@@ -108,4 +130,9 @@
     <child link="left_cliff_sensor_link" />
   </joint>
+  <joint name="base_tray_axis_joint" type="fixed">
+    <origin xyz="0.0 0.0 0.319" rpy="0 1.57079 0" />
+    <parent link="base_link"/>
+    <child link="tray_axis_link" />
+  </joint>
   <joint name="base_right_cliff_sensor_joint" type="fixed">
     <origin xyz="0.07 -0.14 0.01" rpy="0 1.57079 0" />
@@ -229,8 +256,8 @@
     <axis xyz="0 1 0"/>
   </joint>
-  <turtlebot_spacer parent="base_link" number="0" x_loc="-0.00254" y_loc="0.1114679" z_loc="0.062992"/>
-  <turtlebot_spacer parent="base_link" number="1" x_loc="-0.00254" y_loc="-0.1114679" z_loc="0.062992"/>
-  <turtlebot_spacer parent="base_link" number="2" x_loc="-0.07239" y_loc="-0.1114679" z_loc="0.062992"/>
-  <turtlebot_spacer parent="base_link" number="3" x_loc="-0.07239" y_loc="0.1114679" z_loc="0.062992"/>
+  <mobina_spacer parent="base_link" number="0" x_loc="-0.00254" y_loc="0.1114679" z_loc="0.062992"/>
+  <mobina_spacer parent="base_link" number="1" x_loc="-0.00254" y_loc="-0.1114679" z_loc="0.062992"/>
+  <mobina_spacer parent="base_link" number="2" x_loc="-0.07239" y_loc="-0.1114679" z_loc="0.062992"/>
+  <mobina_spacer parent="base_link" number="3" x_loc="-0.07239" y_loc="0.1114679" z_loc="0.062992"/>
   <joint name="gyro_joint" type="fixed">
     <axis xyz="0 1 0" />
@@ -282,5 +309,5 @@
       <origin xyz=" 0 0 0 " rpy="0 0 0" />
       <geometry>
-        <mesh filename="package://turtlebot_description/meshes/plate_0_logo.dae"/>
+        <mesh filename="package://mobina_description/meshes/plate_0_logo.dae"/>
       </geometry>
     </visual>
@@ -292,8 +319,8 @@
     </collision>
   </link>
-  <turtlebot_standoff_2in parent="base_link" number="0" x_loc="0.0676402" y_loc="0.1314196" z_loc="0.0709803"/>
-  <turtlebot_standoff_2in parent="base_link" number="1" x_loc="0.0676402" y_loc="-0.1314196" z_loc="0.0709803"/>
-  <turtlebot_standoff_2in parent="base_link" number="2" x_loc="-0.052832" y_loc="-0.1314196" z_loc="0.0709803"/>
-  <turtlebot_standoff_2in parent="base_link" number="3" x_loc="-0.052832" y_loc="0.1314196" z_loc="0.0709803"/>
+  <mobina_standoff_2in parent="base_link" number="0" x_loc="0.0676402" y_loc="0.1314196" z_loc="0.0709803"/>
+  <mobina_standoff_2in parent="base_link" number="1" x_loc="0.0676402" y_loc="-0.1314196" z_loc="0.0709803"/>
+  <mobina_standoff_2in parent="base_link" number="2" x_loc="-0.052832" y_loc="-0.1314196" z_loc="0.0709803"/>
+  <mobina_standoff_2in parent="base_link" number="3" x_loc="-0.052832" y_loc="0.1314196" z_loc="0.0709803"/>
   <joint name="plate_1_joint" type="fixed">
     <origin xyz="0.04068 0 0.05715" rpy="0 0 0" />
@@ -312,5 +339,5 @@
       <origin xyz=" 0 0 0 " rpy="0 0 0" />
       <geometry>
-        <mesh filename="package://turtlebot_description/meshes/plate_1_logo.dae"/>
+        <mesh filename="package://mobina_description/meshes/plate_1_logo.dae"/>
       </geometry>
     </visual>
@@ -322,8 +349,8 @@
     </collision>
   </link>
-  <turtlebot_standoff_2in parent="standoff_2in_0_link" number="4" x_loc="0" y_loc="0" z_loc="0.05715"/>
-  <turtlebot_standoff_2in parent="standoff_2in_1_link" number="5" x_loc="0" y_loc="0" z_loc="0.05715"/>
-  <turtlebot_standoff_2in parent="standoff_2in_2_link" number="6" x_loc="0" y_loc="0" z_loc="0.05715"/>
-  <turtlebot_standoff_2in parent="standoff_2in_3_link" number="7" x_loc="0" y_loc="0" z_loc="0.05715"/>
+  <mobina_standoff_2in parent="standoff_2in_0_link" number="4" x_loc="0" y_loc="0" z_loc="0.05715"/>
+  <mobina_standoff_2in parent="standoff_2in_1_link" number="5" x_loc="0" y_loc="0" z_loc="0.05715"/>
+  <mobina_standoff_2in parent="standoff_2in_2_link" number="6" x_loc="0" y_loc="0" z_loc="0.05715"/>
+  <mobina_standoff_2in parent="standoff_2in_3_link" number="7" x_loc="0" y_loc="0" z_loc="0.05715"/>
   <joint name="plate_2_joint" type="fixed">
     <origin xyz="0 0 0.0572008" rpy="0 0 0" />
@@ -342,5 +369,5 @@
       <origin xyz=" 0 0 0 " rpy="0 0 0" />
       <geometry>
-        <mesh filename="package://turtlebot_description/meshes/plate_1_logo.dae"/>
+        <mesh filename="package://mobina_description/meshes/plate_1_logo.dae"/>
       </geometry>
     </visual>
@@ -352,10 +379,10 @@
     </collision>
   </link>
-  <turtlebot_standoff_kinect parent="plate_2_link" number="0" x_loc="-0.1024382" y_loc="0.098" z_loc="0.0032004"/>
-  <turtlebot_standoff_kinect parent="plate_2_link" number="1" x_loc="-0.1024382" y_loc="-0.098" z_loc="0.0032004"/>
-  <turtlebot_standoff_8in parent="standoff_2in_4_link" number="0" x_loc="0" y_loc="0" z_loc="0.05715"/>
-  <turtlebot_standoff_8in parent="standoff_2in_5_link" number="1" x_loc="0" y_loc="0" z_loc="0.05715"/>
-  <turtlebot_standoff_8in parent="standoff_2in_6_link" number="2" x_loc="0" y_loc="0" z_loc="0.05715"/>
-  <turtlebot_standoff_8in parent="standoff_2in_7_link" number="3" x_loc="0" y_loc="0" z_loc="0.05715"/>
+  <mobina_standoff_kinect parent="plate_2_link" number="0" x_loc="-0.1024382" y_loc="0.098" z_loc="0.0032004"/>
+  <mobina_standoff_kinect parent="plate_2_link" number="1" x_loc="-0.1024382" y_loc="-0.098" z_loc="0.0032004"/>
+  <mobina_standoff_8in parent="standoff_2in_4_link" number="0" x_loc="0" y_loc="0" z_loc="0.05715"/>
+  <mobina_standoff_8in parent="standoff_2in_5_link" number="1" x_loc="0" y_loc="0" z_loc="0.05715"/>
+  <mobina_standoff_8in parent="standoff_2in_6_link" number="2" x_loc="0" y_loc="0" z_loc="0.05715"/>
+  <mobina_standoff_8in parent="standoff_2in_7_link" number="3" x_loc="0" y_loc="0" z_loc="0.05715"/>
   <joint name="plate_3_joint" type="fixed">
     <origin xyz="-0.01316 0 0.2063496" rpy="0 0 0" />
@@ -374,5 +401,5 @@
       <origin xyz=" 0 0 0 " rpy="0 0 0" />
       <geometry>
-        <mesh filename="package://turtlebot_description/meshes/plate_2_logo.dae"/>
+        <mesh filename="package://mobina_description/meshes/plate_2_logo.dae"/>
       </geometry>
     </visual>
@@ -385,8 +412,8 @@
   </link>
   <!-- Simulation sensors -->
-  <turtlebot_sim_imu/>
-  <turtlebot_sim_laser/>
-  <turtlebot_sim_create/>
-  <turtlebot_sim_wall_sensors/>
+  <mobina_sim_imu/>
+  <mobina_sim_laser/>
+  <mobina_sim_create/>
+  <mobina_sim_wall_sensors/>
   </xacro:macro>
 </robot>

Commit message: fixed gyro link

File: mobina_description/urdf/mobina_body.urdf.xacro (robot description, xacro)
@@ -263,5 +263,5 @@
     <axis xyz="0 1 0" />
     <origin xyz="0 0 0.04" rpy="0 0 0" />
-    <parent link="base_link"/>
+    <parent link="tray_base_link"/>
     <child link="gyro_link"/>
   </joint>

Commit message: added parameter, removed unnecessary parts

File: mobina_description/urdf/mobina_body.urdf.xacro (robot description, xacro)
@@ -4,4 +4,5 @@
   <!-- Macro for mobina body. Including Gazebo extensions, but does not include Kinect -->
   <include filename="$(find mobina_description)/urdf/gazebo.urdf.xacro"/>
+  <include filename="$(find mobina_description)/urdf/mobina_calibration.xacro" />
   <property name="base_x" value="0.33" />
   <property name="base_y" value="0.33" />
@@ -83,4 +84,9 @@
     <child link="tray_base_link"/>
   </joint>
+  <joint name="base_tray_axis_joint" type="fixed">
+    <origin xyz="0.0 0.0 0.319" rpy="${mobina_calib_beta} 1.57079 0" />
+    <parent link="base_link"/>
+    <child link="tray_axis_link" />
+  </joint>
   <link name="left_cliff_sensor_link">
     <inertial>
@@ -129,9 +135,4 @@
     <parent link="base_link"/>
     <child link="left_cliff_sensor_link" />
-  </joint>
-  <joint name="base_tray_axis_joint" type="fixed">
-    <origin xyz="0.0 0.0 0.319" rpy="0 1.57079 0" />
-    <parent link="base_link"/>
-    <child link="tray_axis_link" />
   </joint>
   <joint name="base_right_cliff_sensor_joint" type="fixed">
@@ -293,5 +294,5 @@
     </inertial>
   </link>
-  <joint name="plate_0_joint" type="fixed">
+  <!--joint name="plate_0_joint" type="fixed">
     <origin xyz="-0.04334 0  0.06775704" rpy="0 0 0" />
     <parent link="base_link"/>
@@ -410,5 +411,5 @@
       </geometry>
     </collision>
-  </link>
+  </link-->
   <!-- Simulation sensors -->
   <mobina_sim_imu/>

File: mobina_description/urdf/mobina_calibration.xacro (robot description, xacro)
@@ -5,6 +5,7 @@
   <property name="mobina_calib_cam_z" value="0.105" />
   <property name="mobina_calib_cam_rr" value="0" />
-  <property name="mobina_calib_cam_rp" value="0" />
+  <property name="mobina_calib_cam_rp" value="-1.57079" />
   <property name="mobina_calib_cam_ry" value="0" />
+  <property name="mobina_calib_beta" value="0" />
   <property name="mobina_camera_parent_name" value="tray_base_link" />
 </robot>

Commit message: update to descr.

File: mobina_description/urdf/mobina_body.urdf.xacro (robot description, xacro)
@@ -78,6 +78,6 @@
     </inertial>
   </link>
-  <joint name="tray_axis_joint" type="continuous">
-    <axis xyz="0 1 0"/>
+  <joint name="tray_joint" type="continuous">
+    <axis xyz="0 -1 0"/>
     <origin rpy="0 0 0" xyz="0 0 0"/>
     <parent link="tray_axis_link"/>
@@ -263,5 +263,5 @@
   <joint name="gyro_joint" type="fixed">
     <axis xyz="0 1 0" />
-    <origin xyz="0 0 0.04" rpy="0 0 0" />
+    <origin xyz="0 0 0.04" rpy="-1.57079 0 0" />
     <parent link="tray_base_link"/>
     <child link="gyro_link"/>

Commit message: reusing imu from tablet

File: mobina_description/urdf/mobina_body.urdf.xacro (robot description, xacro)
@@ -261,4 +261,17 @@
   <mobina_spacer parent="base_link" number="2" x_loc="-0.07239" y_loc="-0.1114679" z_loc="0.062992"/>
   <mobina_spacer parent="base_link" number="3" x_loc="-0.07239" y_loc="0.1114679" z_loc="0.062992"/>
+  <!--joint name="gyro_joint" type="fixed">
+    <axis xyz="0 1 0" />
+    <origin xyz="0 0 0.04" rpy="0 0 0" />
+    <parent link="base_link"/>
+    <child link="gyro_link"/>
+  </joint>
+  <link name="gyro_link">
+    <inertial>
+      <mass value="0.001" />
+      <origin xyz="0 0 0" rpy="0 0 0" />
+      <inertia ixx="0.0001" ixy="0" ixz="0" iyy="0.000001" iyz="0" izz="0.0001" />
+    </inertial>
+  </link-->
   <joint name="gyro_joint" type="fixed">
     <axis xyz="0 1 0" />
