Commit message: renaming

File: lcrob1_description/urdf/create.urdf.xacro (robot description, xacro)
@@ -5,5 +5,5 @@
     xmlns:interface="http://playerstage.sourceforge.net/gazebo/xmlschema/#interface">
     <!-- Included URDF Files -->
-    <include filename="$(find irobot_create_description)/urdf/create_base.xacro" />
+    <include filename="$(find lcrob1_description)/urdf/create_base.xacro" />
     <create />
 </robot>

File: lcrob1_description/urdf/create_base.xacro (robot description, xacro)
@@ -5,6 +5,6 @@
     xmlns:interface="http://playerstage.sourceforge.net/gazebo/xmlschema/#interface">
     <!-- Included URDF Files -->
-    <include filename="$(find irobot_create_description)/urdf/materials.urdf.xacro" />
-    <include filename="$(find irobot_create_description)/urdf/create_wheel.xacro" />
+    <include filename="$(find lcrob1_description)/urdf/materials.urdf.xacro" />
+    <include filename="$(find lcrob1_description)/urdf/create_wheel.xacro" />
     <include filename="$(find hector_sensors_description)/urdf/sonar_sensor.urdf.xacro" />
     <!-- Properties (Constants) -->
@@ -63,5 +63,5 @@
                 <origin xyz="0.0 0.0 0.0" rpy="0 0 0" />
                 <geometry>
-                    <mesh filename="package://irobot_create_description/meshes/create_body.dae"/>
+                    <mesh filename="package://lcrob1_description/meshes/create_body.dae"/>
                 </geometry>
                 <material name="Blue" />
@@ -70,5 +70,5 @@
                 <origin xyz="0.0 0.0 0.0" rpy="0 0 0" />
                 <geometry>
-                    <mesh filename="package://irobot_create_description/meshes/create_body.stl"/>
+                    <mesh filename="package://lcrob1_description/meshes/create_body.stl"/>
                 </geometry>
             </collision>
